File: pcb/Bluetooth Mosfet/Bluetooth Mosfet.kicad_sch (KiCad schematic)
At the start: 12 parts, among them J1 1x3 Header, J2 1x4 Header, J3 1x2 Header, J4 1x4 Header, Q1 IRF510N, U2 ATtiny 1614

Commit message: Routed Traces for Milling
Parts:
- D1, D2: footprint (none) -> fab:LED_1206
- R1, R2, R3: footprint (none) -> fab:R_1206
Connections:
- net at J3.1 (Pin_1): now also Q1.2 (D); no longer Q1.S
- net at J3.2 (Pin_2): now also Q1.3 (S); no longer Q1.D
- net at J1.2 (Pin_2), R1.2, R2.2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: now also J2.2 (Pin_2), U2.8 (PB1/SDA); no longer J2.1 (Pin_1)
- net at R3.1, U2.11 (PA1/D8): now also Q1.1 (G); no longer Q1.G
- net at U2.10 (UPDI/PA0/D11): now also J1.1 (Pin_1); no longer J1.3 (Pin_3)
- net at U2.6 (PB3/RXD): now also J2.3 (Pin_3); no longer J2.4 (Pin_4)
- net at U2.7 (PB2/TXD): now also J2.4 (Pin_4); no longer J2.3 (Pin_3)
- new net: J1.3 (Pin_3), J2.1 (Pin_1), U2.1 (VCC)
Other:
- company: (none) -> Nicholas Niles
- title: (none) -> Bluetooth-Controlled Mosfet Board
- moved on the sheet: J3
